File: blinky.kicad_pcb (KiCad board)
At the start: 2 copper layers, 7 parts, among them U1 NA555D

Commit message: Final ordered
Parts:
- BT1: moved to B.Cu
- moved D1 29.2 mm to (102.4, 94.0)
- moved R1 27.3 mm to (86.5, 98.5), turned to 0 degrees
- moved U1 26.6 mm to (95.5, 99.0)
- moved R3 26.0 mm to (102.5, 98.6), turned to 0 degrees
- moved R2 23.5 mm to (90.0, 98.5), turned to 0 degrees
- moved C1 14.0 mm to (100.0, 102.5), turned to 180 degrees
- turned BT1 to 180 degrees
Routing:
- net Net-(U1-THR): track 0.00 -> 12.9 mm
- net GND: track 0.00 -> 6.66 mm, vias 0 -> 2
- net Net-(U1-DIS): track 0.00 -> 6.40 mm
- net VCC: track 0.00 -> 6.08 mm, vias 0 -> 2
- net Net-(D1-A): track 0.00 -> 4.64 mm
- net Net-(U1-Q): track 0.00 -> 4.02 mm
- added copper zone on B.Cu, net GND
- added copper zone on F.Cu, net VCC
Other:
- board outline added: 26.5 x 21 mm
