File: blinky.kicad_sch (KiCad schematic)
At the start: 6 parts, among them U1 NA555D

Commit message: update
Parts:
- added BT1: Battery_Cell, Battery:BatteryHolder_Keystone_3000_1x12mm, symbol Device:Battery_Cell
- C1: footprint (none) -> Capacitor_SMD:C_0402_1005Metric_Pad0.74x0.62mm_HandSolder
- D1: footprint (none) -> LED_SMD:LED_0402_1005Metric_Pad0.77x0.64mm_HandSolder
- R1, R2, R3: footprint (none) -> Resistor_SMD:R_0402_1005Metric_Pad0.72x0.64mm_HandSolder
Connections:
- net GND: now also BT1.2 (-)
- net VCC: now also BT1.1 (+)

Commit message: Final ordered
Other:
- title: (none) -> Blinky
Changed lines of the file:
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@@
 	(generator_version "9.0")
 	(paper "A4")
+	(title_block
+		(title "Blinky")
+		(date "2025-12-25")
+		(rev "1.0")
+	)
 	(junction
 		(at 100.33 125.73)

Commit message: Adding docs
Other:
- company: (none) -> Mitchell McCuiston
Changed lines of the file:
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@@
 		(date "2025-12-25")
 		(rev "1.0")
+		(company "Mitchell McCuiston")
+		(comment 1 "mitch.mcc@gmail.com")
 	)
 	(junction
